Commit message: fix: reset up rviz and add meshes
(not work completely)

File: src/description/urdf/Master.xacro (robot description, xacro)
@@ -2,9 +2,14 @@
 <robot xmlns:xacro="http://www.ros.org/wiki/xacro"  name="Maket">
      <xacro:include filename= "Slave.xacro"/>
-     <link name = "Maket">
+     <link name="dummy"/>
+     <joint name="dummy_to_base_link=" type="fixed">
+          <parent link="dummy"/>
+          <child link="base_link"/>
+     </joint>
+     <link name = "base_link">
           <visual>
                <origin xyz = "0 0 0" rpy = "0 0 0" />
                <geometry>
-                    <mesh filename="package://Maket/meshes/Maket.STL" />
+                    <mesh filename="./ros2_ws/install/description/share/description/meshes/Maket.stl" />
                </geometry>
                <material name="">
@@ -15,5 +20,5 @@
                <origin xyz= "0 0 0" rpy="0 0 0" />
                <geometry>
-                    <mesh filename="package://Maket/meshes/Maket.STL" />
+                    <mesh filename="./ros2_ws/install/description/share/description/meshes/Maket.stl" />
                </geometry>
           </collision>
@@ -38,5 +43,5 @@
                <origin xyz="0 0 0" rpy="0 0 0" />
                <geometry>
-                    <mesh filename="package://Maket/meshes/Right_Wheel.STL"/>
+                    <mesh filename="./ros2_ws/install/description/share/description/meshes/Right_Wheel.stl"/>
                </geometry>
                <material name="Right_Wheel"/>
@@ -45,5 +50,5 @@
                <origin xyz="0 0 0" rpy="0 0 0" />
                <geometry>
-                    <mesh filename="package://Maket/meshes/Right_Wheel.STL"/>
+                    <mesh filename="./ros2_ws/install/description/share/description/meshes/Right_Wheel.stl"/>
                </geometry>
           </collision>
@@ -62,5 +67,5 @@
           />
           <parent
-               link="Maket" />
+               link="base_link" />
           <child
                link="Right_Wheel" />
@@ -80,5 +85,5 @@
                <origin xyz="0 0 0" rpy="0 0 0" />
                <geometry>
-                    <mesh filename="package://Maket/meshes/Left_Wheel.STL"/>
+                    <mesh filename="package://meshes/Left_Wheel.stl"/>
                </geometry>
                <material name="Left_Wheel"/>
@@ -87,5 +92,5 @@
                <origin xyz="0 0 0" rpy="0 0 0" />
                <geometry>
-                    <mesh filename="package://Maket/meshes/Left_Wheel.STL"/>
+                    <mesh filename="package://meshes/Left_Wheel.stl"/>
                </geometry>
           </collision>
@@ -105,5 +110,5 @@
           />
           <parent
-               link="Maket" />
+               link="base_link" />
           <child
                link="Left_Wheel" />
@@ -123,5 +128,5 @@
                <origin xyz="0 0 0" rpy="0 0 0" />
                <geometry>
-                    <mesh filename="package://Maket/meshes/Roller.STL"/>
+                    <mesh filename="package://meshes/Roller.STL"/>
                </geometry>
                <material name="Roller"/>
@@ -130,5 +135,5 @@
                <origin xyz="0 0 0" rpy="0 0 0" />
                <geometry>
-                    <mesh filename="package://Maket/meshes/Roller.STL"/>
+                    <mesh filename="package://meshes/Roller.stl"/>
                </geometry>
           </collision>
@@ -148,5 +153,5 @@
           />
           <parent
-               link="Maket" />
+               link="base_link" />
           <child
                link="Roller" />
