Commit message: Complete first iteration URDF model

File: camera/src/description/urdf/Master.xacro (robot description, xacro)
@@ -11,5 +11,5 @@
                <origin xyz = "0 0 0" rpy = "0 0 0" />
                <geometry>
-                    <mesh filename="./ros2_ws/install/description/share/description/meshes/Maket.stl" />
+                    <mesh filename="package://description/meshes/Maket.stl" />
                </geometry>
                <material name="">
@@ -20,5 +20,5 @@
                <origin xyz= "0 0 0" rpy="0 0 0" />
                <geometry>
-                    <mesh filename="./ros2_ws/install/description/share/description/meshes/Maket.stl" />
+                    <mesh filename="package://description/meshes/Maket.stl" />
                </geometry>
           </collision>
@@ -43,5 +43,5 @@
                <origin xyz="0 0 0" rpy="0 0 0" />
                <geometry>
-                    <mesh filename="./ros2_ws/install/description/share/description/meshes/Right_Wheel.stl"/>
+                    <mesh filename="package://description/meshes/Right_Wheel.stl"/>
                </geometry>
                <material name="Right_Wheel"/>
@@ -50,5 +50,5 @@
                <origin xyz="0 0 0" rpy="0 0 0" />
                <geometry>
-                    <mesh filename="./ros2_ws/install/description/share/description/meshes/Right_Wheel.stl"/>
+                    <mesh filename="package://description/meshes/Right_Wheel.stl"/>
                </geometry>
           </collision>
@@ -85,5 +85,5 @@
                <origin xyz="0 0 0" rpy="0 0 0" />
                <geometry>
-                    <mesh filename="package://meshes/Left_Wheel.stl"/>
+                    <mesh filename="package://description/meshes/Left_Wheel.stl"/>
                </geometry>
                <material name="Left_Wheel"/>
@@ -92,5 +92,5 @@
                <origin xyz="0 0 0" rpy="0 0 0" />
                <geometry>
-                    <mesh filename="package://meshes/Left_Wheel.stl"/>
+                    <mesh filename="package://description/meshes/Left_Wheel.stl"/>
                </geometry>
           </collision>
@@ -106,5 +106,5 @@
      <joint name="LeftWheel" type="continuous">
           <origin
-               xyz="0.040866 -0.2 0.015296"
+               xyz="0.040866 0.2 0.015296"
                rpy="-1.5708 0 0"
           />
@@ -128,5 +128,5 @@
                <origin xyz="0 0 0" rpy="0 0 0" />
                <geometry>
-                    <mesh filename="package://meshes/Roller.STL"/>
+                    <mesh filename="package://description/meshes/Roller.stl"/>
                </geometry>
                <material name="Roller"/>
@@ -135,5 +135,5 @@
                <origin xyz="0 0 0" rpy="0 0 0" />
                <geometry>
-                    <mesh filename="package://meshes/Roller.stl"/>
+                    <mesh filename="package://description/meshes/Roller.stl"/>
                </geometry>
           </collision>

Commit message: Add Odometry and TF (Not completed)

File: camera/src/description/urdf/Master.xacro (robot description, xacro)
@@ -2,9 +2,10 @@
 <robot xmlns:xacro="http://www.ros.org/wiki/xacro"  name="Maket">
      <xacro:include filename= "Slave.xacro"/>
-     <link name="dummy"/>
-     <joint name="dummy_to_base_link=" type="fixed">
-          <parent link="dummy"/>
+     <link name="base_footprint"/>
+     <joint name="base_to_footprint" type="fixed">
+          <parent link="base_footprint"/>
           <child link="base_link"/>
-     </joint>
+          <origin xyz="0 0 0" rpy="0 0 0"/>
+    </joint>
      <link name = "base_link">
           <visual>
