Commit message: complete TF and start navigation stack

File: camera/src/description/urdf/descriptions.xacro (robot description, xacro)
@@ -1,5 +1,5 @@
 <?xml version="1.0"?>
 <robot xmlns:xacro="http://www.ros.org/wiki/xacro"  name="Maket">
-     <xacro:include filename= "Slave.xacro"/>
+     <xacro:include filename= "inertials.xacro"/>
      <link name="base_footprint"/>
      <joint name="base_to_footprint" type="fixed">
@@ -24,18 +24,4 @@
                </geometry>
           </collision>
-          <inertial>
-               <origin
-                    xyz="0.022152700168409 -0.000809996770580155 0.107200331423198"
-                    rpy="0 0 0" />
-               <mass value="2.24483698501812" />
-               <inertia
-                    ixx="0.017171108266307"
-                    ixy="7.41182378513859E-05"
-                    ixz="0.000134548028700423"
-                    iyy="0.00556240946464024"
-                    iyz="-8.46684644335415E-05"
-                    izz="0.0154086578851944"
-               />
-          </inertial>
      </link>
      <!-- <Right_Wheel> -->
@@ -54,16 +40,9 @@
                </geometry>
           </collision>
-          <!-- <inertial> -->
-          <xacro:Right_Wheel mass="0.0609278440646647">
-               <origin
-                    xyz="-6.175795070019E-18 -2.42861286636753E-17 0.0116563539649974"
-                    rpy="0 0 0" />
-          </xacro:Right_Wheel>
-          <!-- <inertial/> -->
      </link>
      <joint name="RightWheel" type="continuous">
           <origin
                xyz="0.040866 -0.2 0.015296"
-               rpy="-1.5708 0 0"
+               rpy="1.5708 0 0"
           />
           <parent
@@ -73,10 +52,10 @@
           <axis
                xyz="0 0 1" />
-          <limit
+          <!-- <limit
                effort="10"
-               velocity="10" />
-          <dynamics
+               velocity="10" /> -->
+          <!-- <dynamics
                damping="0.1"
-               friction="0.1" />
+               friction="0.1" /> -->
      </joint>
      <!-- </Right_Wheel> -->
@@ -96,12 +75,4 @@
                </geometry>
           </collision>
-          <!-- <inertial> -->
-          <xacro:Left_Wheel mass="0.0577108531873887">
-               <origin
-                    xyz="-2.26065295916128E-19 -2.42861286636753E-17 -0.010522332891134"
-                    rpy="0 0 0"
-               />
-          </xacro:Left_Wheel>
-          <!-- <inertial/> -->
      </link>
      <joint name="LeftWheel" type="continuous">
@@ -116,10 +87,10 @@
           <axis
                xyz="0 0 1" />
-          <limit
+          <!-- <limit
                effort="10"
                velocity="10" />
           <dynamics
                damping="0.1"
-               friction="0.1" />
+               friction="0.1" /> -->
      </joint>
      <!--</Left_Whell>-->
@@ -139,12 +110,4 @@
                </geometry>
           </collision>
-          <!-- <inertial> -->
-          <xacro:Roller mass="0.0106249291862938">
-          <origin
-               xyz="0 -2.16840434497101E-19 -1.24564498913758E-18"
-               rpy="0 0 0"
-          />
-          </xacro:Roller>
-          <!-- <inertial/> -->
      </link>
      <joint name="Roller" type="continuous">
@@ -159,10 +122,10 @@
           <axis
                xyz="0 0 -1" />
-          <limit
+          <!-- <limit
                effort="10"
                velocity="10" />
           <dynamics
                damping="0.1"
-               friction="0.1" />
+               friction="0.1" /> -->
      </joint>
      <!--</Roller>-->

File: camera/src/description/urdf/inertials.xacro (robot description, xacro)
@@ -3,9 +3,4 @@
     <!-- This file is not a robot in and of itself, it just contains some useful tags that could be included in any robot -->
     <!-- Specify some colours -->
-    <!--<material name="Maket">
-        <color
-          rgba="1 0.898039215686275 0.8 1" />
-      </material>
--->
     <material name="Right_Wheel">
         <color
@@ -22,20 +17,21 @@
     <!-- Specify some standard inertial calculations https://en.wikipedia.org/wiki/List_of_moments_of_inertia -->
     <!-- These make use of xacro's mathematical functionality -->
-<!--
-    <xacro:macro name = "Maket" params = "mass *origin">
+    <!-- <base_link> -->
+    <!-- <xacro:macro name = "base_link" params = "mass *origin">
         <inertial>
-            <xacro:insert_block name="origin"/>
-            <mass value="${mass}" />
-            <inertia
-                ixx="0.017171108266307"
-                ixy="7.41182378513859E-05"
-                ixz="0.000134548028700423"
-                iyy="0.00556240946464024"
-                iyz="-8.46684644335415E-05"
-                izz="0.0154086578851944"
-            />
-        </inertial>
-    </xacro:macro>
-    -->
+               <origin
+                    xyz="0.022152700168409 -0.000809996770580155 0.107200331423198"
+                    rpy="0 0 0" />
+               <mass value="2.24483698501812" />
+               <inertia
+                    ixx="0.017171108266307"
+                    ixy="7.41182378513859E-05"
+                    ixz="0.000134548028700423"
+                    iyy="0.00556240946464024"
+                    iyz="-8.46684644335415E-05"
+                    izz="0.0154086578851944"
+               />
+          </inertial>
+    </xacro:macro> -->
     <!-- <Right_Wheel> -->
     <xacro:macro name = "Right_Wheel" params = "mass *origin">

File: camera/src/description/urdf/robot.urdf.xacro (robot description, xacro)
@@ -1,4 +1,4 @@
 <?xml version="1.0"?>
 <robot xmlns:xacro="http://www.ros.org/wiki/xacro"  name="Maket">
-    <xacro:include filename="Master.xacro"/>
+    <xacro:include filename="descriptions.xacro"/>
 </robot>

Commit message: feat(SLAM): Prepare urdf to lidar launch

File: camera/src/description/urdf/descriptions.xacro (robot description, xacro)
@@ -2,5 +2,5 @@
 <robot xmlns:xacro="http://www.ros.org/wiki/xacro"  name="Maket">
      <xacro:include filename= "inertials.xacro"/>
-     <xacro:include filename= "sensors.xacro"/>
+     <xacro:include filename= "sensors.urdf.xacro"/>
      <link name="base_footprint"/>
      <joint name="base_to_footprint" type="fixed">
@@ -131,4 +131,21 @@
      </joint>
      <!--</Roller>-->
-      <xacro:imu/>
+     <xacro:imu/>
+     <xacro:generic_laser>
+          <xacro:macro name="generic_laser" params="*origin">
+          <xacro:laser
+               update_rate="10"
+               ray_count="360"
+               min_angle="-3.1416"
+               max_angle="3.1416"
+               min_range="0.08"
+               max_range="12.0"
+               frame_id="laser"
+               topic_name="scan"
+          >
+               <xacro:insert_block name="origin" />
+          </xacro:laser>
+          </xacro:macro>
+          <xacro:insert_block name="laser_pose" />
+     </xacro:generic_laser>
 </robot>

Commit message: feat(SLAM): Add lidar model to URDF

File: camera/src/description/urdf/descriptions.xacro (robot description, xacro)
@@ -132,20 +132,6 @@
      <!--</Roller>-->
      <xacro:imu/>
-     <xacro:generic_laser>
-          <xacro:macro name="generic_laser" params="*origin">
-          <xacro:laser
-               update_rate="10"
-               ray_count="360"
-               min_angle="-3.1416"
-               max_angle="3.1416"
-               min_range="0.08"
-               max_range="12.0"
-               frame_id="laser"
-               topic_name="scan"
-          >
-               <xacro:insert_block name="origin" />
-          </xacro:laser>
-          </xacro:macro>
-          <xacro:insert_block name="laser_pose" />
-     </xacro:generic_laser>
+     <xacro:laser>
+          <origin xyz="0 0 0.33" rpy="0 0 0"/>
+     </xacro:laser>
 </robot>

File: camera/src/description/urdf/sensors.urdf.xacro (robot description, xacro)
@@ -1,2 +1,3 @@
+<?xml version="1.0"?>
 <robot xmlns:xacro="http://ros.org/wiki/xacro">
   <xacro:macro name="imu">
@@ -9,5 +10,5 @@
   </xacro:macro>
   <xacro:macro name="laser" params="*origin">
-    <link name="${frame_id}">
+    <link name="lidar">
       <visual>
         <origin xyz="0 0 -0.025" rpy="0 0 0"/>
@@ -25,9 +26,17 @@
         </geometry>
       </collision>
-      <joint name="${frame_id}_to_base_link" type="fixed">
-        <parent link="base_link"/>
-        <child link="${frame_id}"/>
-        <xacro:insert_block name="origin" />
-      </joint>
-    </xacro:macro>
+      <inertial>
+        <origin xyz="0 0 0" rpy="0 0 0"/>
+        <mass value="0.1"/>
+        <inertia ixx="${(2/5) * 0.1 * (0.0375 * 0.0375)}" ixy="0" ixz="0"
+                 iyy="${(2/5) * 0.1 * (0.0375 * 0.0375)}" iyz="0"
+                 izz="${(2/5) * 0.1 * (0.0375 * 0.0375)}" />
+      </inertial>
+    </link>
+    <joint name="lidar_to_base_link" type="fixed">
+      <parent link="base_link"/>
+      <child link="lidar"/>
+      <xacro:insert_block name="origin" />
+    </joint>
+  </xacro:macro>
 </robot>
