Commit message: feat: smth done

File: src/ros2/description/urdf/descriptions.xacro (robot description, xacro)
@@ -1,15 +1,15 @@
 <?xml version="1.0"?>
-<robot xmlns:xacro="http://www.ros.org/wiki/xacro"  name="Maket">
-     <xacro:include filename= "inertials.xacro"/>
-     <xacro:include filename= "sensors.urdf.xacro"/>
-     <link name="base_footprint"/>
+<robot xmlns:xacro="http://www.ros.org/wiki/xacro" name="Maket">
+     <xacro:include filename="inertials.xacro" />
+     <xacro:include filename="sensors.urdf.xacro" />
+     <link name="base_footprint" />
      <joint name="base_to_footprint" type="fixed">
-          <parent link="base_footprint"/>
-          <child link="base_link"/>
-          <origin xyz="0 0 0" rpy="0 0 0"/>
-    </joint>
-     <link name = "base_link">
+          <parent link="base_footprint" />
+          <child link="base_link" />
+          <origin xyz="0 0 0" rpy="0 0 0" />
+     </joint>
+     <link name="base_link">
           <visual>
-               <origin xyz = "0 0 0" rpy = "0 0 0" />
+               <origin xyz="0 0 0" rpy="0 0 0" />
                <geometry>
                     <mesh filename="package://description/meshes/Maket.stl" />
@@ -20,5 +20,5 @@
           </visual>
           <collision>
-               <origin xyz= "0 0 0" rpy="0 0 0" />
+               <origin xyz="0 0 0" rpy="0 0 0" />
                <geometry>
                     <mesh filename="package://description/meshes/Maket.stl" />
@@ -31,12 +31,12 @@
                <origin xyz="0 0 0" rpy="0 0 0" />
                <geometry>
-                    <mesh filename="package://description/meshes/Right_Wheel.stl"/>
+                    <mesh filename="package://description/meshes/Right_Wheel.stl" />
                </geometry>
-               <material name="Right_Wheel"/>
+               <material name="Right_Wheel" />
           </visual>
           <collision>
                <origin xyz="0 0 0" rpy="0 0 0" />
                <geometry>
-                    <mesh filename="package://description/meshes/Right_Wheel.stl"/>
+                    <mesh filename="package://description/meshes/Right_Wheel.stl" />
                </geometry>
           </collision>
@@ -66,12 +66,12 @@
                <origin xyz="0 0 0" rpy="0 0 0" />
                <geometry>
-                    <mesh filename="package://description/meshes/Left_Wheel.stl"/>
+                    <mesh filename="package://description/meshes/Left_Wheel.stl" />
                </geometry>
-               <material name="Left_Wheel"/>
+               <material name="Left_Wheel" />
           </visual>
           <collision>
                <origin xyz="0 0 0" rpy="0 0 0" />
                <geometry>
-                    <mesh filename="package://description/meshes/Left_Wheel.stl"/>
+                    <mesh filename="package://description/meshes/Left_Wheel.stl" />
                </geometry>
           </collision>
@@ -101,12 +101,12 @@
                <origin xyz="0 0 0" rpy="0 0 0" />
                <geometry>
-                    <mesh filename="package://description/meshes/Roller.stl"/>
+                    <mesh filename="package://description/meshes/Roller.stl" />
                </geometry>
-               <material name="Roller"/>
+               <material name="Roller" />
           </visual>
           <collision>
                <origin xyz="0 0 0" rpy="0 0 0" />
                <geometry>
-                    <mesh filename="package://description/meshes/Roller.stl"/>
+                    <mesh filename="package://description/meshes/Roller.stl" />
                </geometry>
           </collision>
@@ -123,15 +123,31 @@
           <axis
                xyz="0 0 -1" />
-          <!-- <limit
-               effort="10"
-               velocity="10" />
-          <dynamics
-               damping="0.1"
-               friction="0.1" /> -->
      </joint>
      <!--</Roller>-->
-     <xacro:imu/>
+     <xacro:imu />
      <xacro:laser>
-          <origin xyz="0 0 0.33" rpy="0 0 0"/>
+          <origin xyz="0 0 0.33" rpy="0 0 0" />
      </xacro:laser>
+     <link name="aruco">
+          <visual>
+               <origin xyz="0 0 0" rpy="0 0 0" />
+               <geometry>
+                    <box size="0.10 0.10 0.02" />
+               </geometry>
+               <material name="blue">
+                    <color rgba="0 0 1 1.0" />
+               </material>
+          </visual>
+          <collision>
+               <origin xyz="0 0 0" rpy="0 0 0" />
+               <geometry>
+                    <box size="0.10 0.10 0.02" />
+               </geometry>
+          </collision>
+     </link>
+     <joint name="aruco" type="fixed">
+          <parent link="base_link" />
+          <child link="aruco" />
+          <origin xyz="-0.09 0 0.26" rpy="0 0 0" />
+     </joint>
 </robot>

File: src/ros2/description/urdf/sensors.urdf.xacro (robot description, xacro)
@@ -6,5 +6,5 @@
       <parent link="base_link"/>
       <child link="imu_link"/>
-      <origin xyz="0 0 0" rpy="0 0 0"/>
+      <origin xyz="0 0 0" rpy="3.14 0 0"/>
     </joint>
   </xacro:macro>

Commit message: Correct URDF push

File: src/ros2/description/urdf/descriptions.xacro (robot description, xacro)
@@ -1,4 +1,4 @@
-<?xml version="1.0"?>
-<robot xmlns:xacro="http://www.ros.org/wiki/xacro" name="Maket">
+<?xml version="1.0" encoding="utf-8"?>
+<robot xmlns:xacro="http://www.ros.org/wiki/xacro"  name="Maket">
      <xacro:include filename="inertials.xacro" />
      <xacro:include filename="sensors.urdf.xacro" />
@@ -9,41 +9,45 @@
           <origin xyz="0 0 0" rpy="0 0 0" />
      </joint>
-     <link name="base_link">
+     <link name = "base_link">
           <visual>
-               <origin xyz="0 0 0" rpy="0 0 0" />
+               <origin xyz = "0 0 0" rpy = "0 0 0" />
                <geometry>
-                    <mesh filename="package://description/meshes/Maket.stl" />
+                    <mesh filename="package://Maket/meshes/base_link.STL" />
                </geometry>
-               <material name="">
-                    <color rgba="1 0.898039215686275 0.8 1" />
-               </material>
+               <material name="Maket">
           </visual>
           <collision>
-               <origin xyz="0 0 0" rpy="0 0 0" />
+               <origin xyz= "0 0 0" rpy="0 0 0" />
                <geometry>
-                    <mesh filename="package://description/meshes/Maket.stl" />
+                    <mesh filename="package://Maket/meshes/base_link.STL" />
                </geometry>
           </collision>
+          <!-- <inertial> -->
+          <xacro:Maket mass = "4"/>
+          <!-- <inertial/> -->
      </link>
      <!-- <Right_Wheel> -->
-     <link name="Right_Wheel">
+     </link name = "Right_Wheel">
           <visual>
-               <origin xyz="0 0 0" rpy="0 0 0" />
+               <origin xyz = "0 0 0" rpy = "0 0 0" />
                <geometry>
-                    <mesh filename="package://description/meshes/Right_Wheel.stl" />
+                    <mesh filename = "package://Maket/meshes/right_wheel.STL"/>
                </geometry>
-               <material name="Right_Wheel" />
+               <material name = "Right_Wheel"/>
           </visual>
           <collision>
-               <origin xyz="0 0 0" rpy="0 0 0" />
+               <origin xyz = "0 0 0" rpy = "0 0 0" />
                <geometry>
-                    <mesh filename="package://description/meshes/Right_Wheel.stl" />
+                    <mesh filename = "package://Maket/meshes/right_wheel.STL"/>
                </geometry>
           </collision>
+          <!-- <inertial> -->
+          <xaccro:Right_Wheel mass = "0.077714"/>
+          <!-- <inertial/> -->
      </link>
      <joint name="RightWheel" type="continuous">
           <origin
-               xyz="0.040866 -0.2 0.015296"
-               rpy="1.5708 0 0"
+               xyz="0.059148 -0.2 0.021"
+               rpy="-1.5708 0 0"
           />
           <parent
@@ -53,31 +57,34 @@
           <axis
                xyz="0 0 1" />
-          <!-- <limit
+          <limit
                effort="10"
-               velocity="10" /> -->
-          <!-- <dynamics
+               velocity="10" />
+          <dynamics
                damping="0.1"
-               friction="0.1" /> -->
+               friction="0.1" />
      </joint>
      <!-- </Right_Wheel> -->
      <!-- <Left_Wheel> -->
-     <link name="Left_Wheel">
+     </link name = "Left_Wheel">
           <visual>
-               <origin xyz="0 0 0" rpy="0 0 0" />
+               <origin xyz = "0 0 0" rpy = "0 0 0" />
                <geometry>
-                    <mesh filename="package://description/meshes/Left_Wheel.stl" />
+                    <mesh filename = "package://Maket/meshes/left_wheel.STL"/>
                </geometry>
-               <material name="Left_Wheel" />
+               <material name = "Left_Wheel"/>
           </visual>
           <collision>
-               <origin xyz="0 0 0" rpy="0 0 0" />
+               <origin xyz = "0 0 0" rpy = "0 0 0" />
                <geometry>
-                    <mesh filename="package://description/meshes/Left_Wheel.stl" />
+                    <mesh filename = "package://Maket/meshes/left_wheel.STL"/>
                </geometry>
           </collision>
+          <!-- <inertial> -->
+          <xaccro:Left_Wheel mass = "0.077714"/>
+          <!-- <inertial/> -->
      </link>
      <joint name="LeftWheel" type="continuous">
           <origin
-               xyz="0.040866 0.2 0.015296"
+               xyz="0.059148 0.2 0.021"
                rpy="-1.5708 0 0"
           />
@@ -88,41 +95,12 @@
           <axis
                xyz="0 0 1" />
-          <!-- <limit
+          <limit
                effort="10"
                velocity="10" />
           <dynamics
                damping="0.1"
-               friction="0.1" /> -->
+               friction="0.1" />
      </joint>
      <!--</Left_Whell>-->
-     <!-- <Roller> -->
-     <link name="Roller">
-          <visual>
-               <origin xyz="0 0 0" rpy="0 0 0" />
-               <geometry>
-                    <mesh filename="package://description/meshes/Roller.stl" />
-               </geometry>
-               <material name="Roller" />
-          </visual>
-          <collision>
-               <origin xyz="0 0 0" rpy="0 0 0" />
-               <geometry>
-                    <mesh filename="package://description/meshes/Roller.stl" />
-               </geometry>
-          </collision>
-     </link>
-     <joint name="Roller" type="continuous">
-          <origin
-               xyz="-0.055737 0 -0.005"
-               rpy="-1.5708 0 0"
-          />
-          <parent
-               link="base_link" />
-          <child
-               link="Roller" />
-          <axis
-               xyz="0 0 -1" />
-     </joint>
-     <!--</Roller>-->
      <xacro:imu />
      <xacro:laser>

File: src/ros2/description/urdf/inertials.xacro (robot description, xacro)
@@ -1,84 +1,77 @@
-<?xml version="1.0"?>
+<?xml version="1.0" encoding="utf-8"?>
 <robot xmlns:xacro="http://www.ros.org/wiki/xacro" >
     <!-- This file is not a robot in and of itself, it just contains some useful tags that could be included in any robot -->
     <!-- Specify some colours -->
+    <material name="Maket">
+        <color
+          rgba="1.0 0.1 0.1 1.0" />
+      </material>
     <material name="Right_Wheel">
         <color
-          rgba="1 0.6 0.2 1" />
+          rgba="0.1 0.1 1.0 1.0" />
       </material>
     <material name="Left_Wheel">
         <color
-          rgba="1 0.6 0.2 1" />
-      </material>
-    <material name="Roller">
-        <color
-          rgba="1 0.6 0.2 1" />
+          rgba="0.1 0.1 1.0 1.0" />
       </material>
     <!-- Specify some standard inertial calculations https://en.wikipedia.org/wiki/List_of_moments_of_inertia -->
     <!-- These make use of xacro's mathematical functionality -->
-    <!-- <base_link> -->
-    <!-- <xacro:macro name = "base_link" params = "mass *origin">
+    <xacro:macro name="base_link" params="mass *origin">
         <inertial>
-               <origin
-                    xyz="0.022152700168409 -0.000809996770580155 0.107200331423198"
-                    rpy="0 0 0" />
-               <mass value="2.24483698501812" />
-               <inertia
-                    ixx="0.017171108266307"
-                    ixy="7.41182378513859E-05"
-                    ixz="0.000134548028700423"
-                    iyy="0.00556240946464024"
-                    iyz="-8.46684644335415E-05"
-                    izz="0.0154086578851944"
-               />
-          </inertial>
-    </xacro:macro> -->
+            <xacro:insert_block name="origin"/>
+            <mass value="${mass}" />
+            <inertia
+                ixx="0.013117"
+                ixy="0.00012016"
+                ixz="0.00018351"
+                iyy="0.0036472"
+                iyz="-0.00011926"
+                izz="0.012625"
+            />
+        </inertial>
+        <origin
+            xyz="0.045317 0.00098805 0.11116"
+            rpy="0 0 0"
+        />
+    </xacro:macro>
     <!-- <Right_Wheel> -->
-    <xacro:macro name = "Right_Wheel" params = "mass *origin">
+    <xacro:Macro name = "Right_Wheel" params = "mass *origin">
         <inertial>
             <xacro:insert_block name = "origin"/>
             <mass value = "${mass}"/>
             <inertia
-                ixx="1.61548368325699E-05"
-                ixy="2.20581496687333E-25"
-                ixz="5.46368876626065E-22"
-                iyy="1.61548368325699E-05"
-                iyz="-8.00640302327215E-21"
-                izz="2.55932138713017E-05"
+                ixx="3.6651E-05"
+                ixy="1.1064E-20"
+                ixz="1.0295E-19"
+                iyy="3.6651E-05"
+                iyz="2.3912E-21"
+                izz="5.4175E-05"
             />
         </inertial>
-    </xacro:macro>
+        <origin
+            xyz="7.9797E-17 -3.4694E-18 0.013353"
+            rpy="0 0 0"
+        />
+    </xacro:Macro>
     <!-- </Right_Wheel> -->
     <!-- <Left_Wheel> -->
-    <xacro:macro name = "Left_Wheel" params = "mass *origin">
+    <xacro:Macro name = "Left_Wheel" params = "mass *origin">
         <inertial>
             <xacro:insert_block name = "origin"/>
             <mass value = "${mass}"/>
             <inertia
-                ixx="1.50439026496173E-05"
-                ixy="3.8344358952925E-24"
-                ixz="-7.45264249140294E-23"
-                iyy="1.50439026496173E-05"
-                iyz="1.07315574491882E-20"
-                izz="2.55674779442835E-05"
+                ixx="3.6651E-05"
+                ixy="-1.3584E-21"
+                ixz="-9.0384E-18"
+                iyy="3.6651E-05"
+                iyz="7.1785E-19"
+                izz="5.4175E-05"
             />
         </inertial>
-    </xacro:macro>
+        <origin
+            xyz="6.8834E-15 -5.5164E-16 -0.013353"
+            rpy="0 0 0"
+        />
+    </xacro:Macro>
     <!-- </Left_Wheel> -->
-    <!-- <Roller_Wheel> -->
-    <xacro:macro name = "Roller" params = "mass *origin">
-        <inertial>
-            <xacro:insert_block name = "origin"/>
-            <mass value = "${mass}"/>
-            <inertia
-                ixx="1.45256797391153E-06"
-                ixy="2.30645963814273E-39"
-                ixz="1.03955497655845E-24"
-                iyy="1.45256797391153E-06"
-                iyz="-1.31736089733523E-22"
-                izz="5.42471410392509E-07"
-            />
-        </inertial>
-    </xacro:macro>
-    <!-- </Roller_Wheel> -->
 </robot>

Commit message: Xacro:macro modified: structure, sensors

File: src/ros2/description/urdf/descriptions.xacro (robot description, xacro)
@@ -1,6 +1,6 @@
 <?xml version="1.0" encoding="utf-8"?>
 <robot xmlns:xacro="http://www.ros.org/wiki/xacro"  name="Maket">
-     <xacro:include filename="inertials.xacro" />
-     <xacro:include filename="sensors.urdf.xacro" />
+     <xacro:include filename="structure.xacro" />
+     <xacro:include filename="sensors.xacro" />
      <link name="base_footprint" />
      <joint name="base_to_footprint" type="fixed">
@@ -9,123 +9,104 @@
           <origin xyz="0 0 0" rpy="0 0 0" />
      </joint>
-     <link name = "base_link">
-          <visual>
-               <origin xyz = "0 0 0" rpy = "0 0 0" />
-               <geometry>
-                    <mesh filename="package://Maket/meshes/base_link.STL" />
-               </geometry>
-               <material name="Maket">
-          </visual>
-          <collision>
-               <origin xyz= "0 0 0" rpy="0 0 0" />
-               <geometry>
-                    <mesh filename="package://Maket/meshes/base_link.STL" />
-               </geometry>
-          </collision>
-          <!-- <inertial> -->
-          <xacro:Maket mass = "4"/>
-          <!-- <inertial/> -->
-     </link>
+     <xacro:base_link name="base_link" mass="5">
+          <origin
+               xyz="0.055795 0.00111 0.11345"
+               rpy="0 0 0"
+          />
+          <inertia
+               ixx="0.01219"
+               ixy="0.00012117"
+               ixz="0.00018358"
+               iyy="0.0027513"
+               iyz="-0.00011927"
+               izz="0.012455"
+          />
+     </xacro:base_link>
      <!-- <Right_Wheel> -->
-     </link name = "Right_Wheel">
-          <visual>
-               <origin xyz = "0 0 0" rpy = "0 0 0" />
-               <geometry>
-                    <mesh filename = "package://Maket/meshes/right_wheel.STL"/>
-               </geometry>
-               <material name = "Right_Wheel"/>
-          </visual>
-          <collision>
-               <origin xyz = "0 0 0" rpy = "0 0 0" />
-               <geometry>
-                    <mesh filename = "package://Maket/meshes/right_wheel.STL"/>
-               </geometry>
-          </collision>
-          <!-- <inertial> -->
-          <xaccro:Right_Wheel mass = "0.077714"/>
-          <!-- <inertial/> -->
-     </link>
-     <joint name="RightWheel" type="continuous">
+     <xacro:wheel_link
+          name_link="right_wheel"
+          filename="package://Макет/meshes/right_wheel.STL"
+          mass="0.08" >
+          <origin
+               xyz="8.3267E-17 0 0.013353"
+               rpy="0 0 0"
+          />
+          <inertia
+               ixx="3.6651E-05"
+               ixy="1.1089E-20"
+               ixz="1.0295E-19"
+               iyy="3.6651E-05"
+               iyz="2.2675E-21"
+               izz="5.4175E-05"
+          />
+     </xacro:wheel_link>
+     <xacro:wheel_joint
+          name="rightwheel"
+          name_link ="right_wheel">
           <origin
                xyz="0.059148 -0.2 0.021"
                rpy="-1.5708 0 0"
           />
-          <parent
-               link="base_link" />
-          <child
-               link="Right_Wheel" />
-          <axis
-               xyz="0 0 1" />
-          <limit
-               effort="10"
-               velocity="10" />
-          <dynamics
-               damping="0.1"
-               friction="0.1" />
-     </joint>
+     </xacro:wheel_joint>
      <!-- </Right_Wheel> -->
      <!-- <Left_Wheel> -->
-     </link name = "Left_Wheel">
-          <visual>
-               <origin xyz = "0 0 0" rpy = "0 0 0" />
-               <geometry>
-                    <mesh filename = "package://Maket/meshes/left_wheel.STL"/>
-               </geometry>
-               <material name = "Left_Wheel"/>
-          </visual>
-          <collision>
-               <origin xyz = "0 0 0" rpy = "0 0 0" />
-               <geometry>
-                    <mesh filename = "package://Maket/meshes/left_wheel.STL"/>
-               </geometry>
-          </collision>
-          <!-- <inertial> -->
-          <xaccro:Left_Wheel mass = "0.077714"/>
-          <!-- <inertial/> -->
-     </link>
-     <joint name="LeftWheel" type="continuous">
+     <xacro:wheel_link
+          name_link="left_wheel"
+          filename="package://Макет/meshes/left_wheel.STL"
+          mass="0.08" >
           <origin
-               xyz="0.059148 0.2 0.021"
+               xyz="3.8886E-14 3.645E-14 0.38665"
+               rpy="0 0 0"
+          />
+          <inertia
+               ixx="3.6651E-05"
+               ixy="-1.2633E-21"
+               ixz="-9.0385E-18"
+               iyy="3.6651E-05"
+               iyz="7.177E-19"
+               izz="5.4175E-05"
+          />
+     </xacro:wheel_link>
+     <xacro:wheel_joint
+          name="leftwheel"
+          name_link="left_wheel">
+          <origin
+               xyz="0.059148 -0.2 0.021"
                rpy="-1.5708 0 0"
           />
-          <parent
-               link="base_link" />
-          <child
-               link="Left_Wheel" />
-          <axis
-               xyz="0 0 1" />
-          <limit
-               effort="10"
-               velocity="10" />
-          <dynamics
-               damping="0.1"
-               friction="0.1" />
-     </joint>
-     <!--</Left_Whell>-->
-     <xacro:imu />
-     <xacro:laser>
-          <origin xyz="0 0 0.33" rpy="0 0 0" />
-     </xacro:laser>
-     <link name="aruco">
-          <visual>
-               <origin xyz="0 0 0" rpy="0 0 0" />
-               <geometry>
-                    <box size="0.10 0.10 0.02" />
-               </geometry>
-               <material name="blue">
-                    <color rgba="0 0 1 1.0" />
-               </material>
-          </visual>
-          <collision>
-               <origin xyz="0 0 0" rpy="0 0 0" />
-               <geometry>
-                    <box size="0.10 0.10 0.02" />
-               </geometry>
-          </collision>
-     </link>
-     <joint name="aruco" type="fixed">
-          <parent link="base_link" />
-          <child link="aruco" />
+     </xacro:wheel_joint>
+     <!-- <Left_Wheel> -->
+     <!-- <IMU> -->
+     <xacro:imu/>
+     <!-- <IMU> -->
+     <!-- <Lidar> -->
+     <xacro:lidar_link
+          filename="package://Макет/meshes/lidar_link.STL"
+          mass = "0.25" >
+          <origin
+               xyz="0.00012979 -6.6734E-06 -0.0079009"
+               rpy="0 0 0"
+          />
+          <inertia
+               ixx="9.5253E-06"
+               ixy="6.45E-11"
+               ixz="4.1315E-08"
+               iyy="9.4166E-06"
+               iyz="6.3454E-09"
+               izz="1.7083E-05"
+          />
+     </xacro:lidar_link>
+     <xacro:lidar_joint>
+          <origin
+               xyz="0.005563 0.002859 0.30015"
+               rpy="0 0 0"
+          />
+     </xacro:lidar_joint>
+     <!-- <Lidar> -->
+     <!-- <Aruco> -->
+     <xacro:aruco>
+          <box size="0.10 0.10 0.02" />
           <origin xyz="-0.09 0 0.26" rpy="0 0 0" />
-     </joint>
+     </xacro:aruco>
+     <!-- <Aruco> -->
 </robot>
