Commit message: meshes fix

File: src/ros2/description/urdf/descriptions.xacro (robot description, xacro)
@@ -9,5 +9,5 @@
           <origin xyz="0 0 0" rpy="0 0 0" />
      </joint>
-     <xacro:base_link name="base_link" mass="5">
+     <xacro:base_link name="base_lnk" mass="5" filename="//description/meshes/base_link.STL">
           <origin
                xyz="0.055795 0.00111 0.11345"
@@ -26,5 +26,5 @@
      <xacro:wheel_link
           name_link="right_wheel"
-          filename="package://Макет/meshes/right_wheel.STL"
+          filename="package://description/meshes/right_wheel.STL"
           mass="0.08" >
           <origin
@@ -53,5 +53,5 @@
      <xacro:wheel_link
           name_link="left_wheel"
-          filename="package://Макет/meshes/left_wheel.STL"
+          filename="package://description/meshes/left_wheel.STL"
           mass="0.08" >
           <origin
@@ -82,5 +82,5 @@
      <!-- <Lidar> -->
      <xacro:lidar_link
-          filename="package://Макет/meshes/lidar_link.STL"
+          filename="package://description/meshes/lidar_link.STL"
           mass = "0.25" >
           <origin

File: src/ros2/description/urdf/structure.xacro (robot description, xacro)
@@ -15,5 +15,5 @@
     </material>
     <!-- Macros for base_link-->
-    <xacro:macro name="base_link" params="name mass *origin *inertia">
+    <xacro:macro name="base_link" params="name mass filename *origin *inertia">
         <link name = "${name}">
             <visual>
@@ -23,5 +23,5 @@
                 />
                 <geometry>
-                    <mesh filename="package://Макет/meshes/base_link.STL" />
+                    <mesh filename="${filename}" />
                 </geometry>
                 <material name="base_link" />

Commit message: almost fine xacro - odom error

File: src/ros2/description/urdf/descriptions.xacro (robot description, xacro)
@@ -1,4 +1,4 @@
 <?xml version="1.0" encoding="utf-8"?>
-<robot xmlns:xacro="http://www.ros.org/wiki/xacro"  name="Maket">
+<robot xmlns:xacro="http://www.ros.org/wiki/xacro">
      <xacro:include filename="structure.xacro" />
      <xacro:include filename="sensors.xacro" />
@@ -9,5 +9,8 @@
           <origin xyz="0 0 0" rpy="0 0 0" />
      </joint>
-     <xacro:base_link name="base_lnk" mass="5" filename="//description/meshes/base_link.STL">
+     <xacro:base_m
+          name="base_link"
+          mass="5"
+          filename="package://description/meshes/base_link.STL">
           <origin
                xyz="0.055795 0.00111 0.11345"
@@ -22,10 +25,10 @@
                izz="0.012455"
           />
-     </xacro:base_link>
+     </xacro:base_m>
      <!-- <Right_Wheel> -->
      <xacro:wheel_link
           name_link="right_wheel"
           filename="package://description/meshes/right_wheel.STL"
-          mass="0.08" >
+          mass="0.08">
           <origin
                xyz="8.3267E-17 0 0.013353"
@@ -43,5 +46,5 @@
      <xacro:wheel_joint
           name="rightwheel"
-          name_link ="right_wheel">
+          name_link="right_wheel">
           <origin
                xyz="0.059148 -0.2 0.021"
@@ -54,5 +57,5 @@
           name_link="left_wheel"
           filename="package://description/meshes/left_wheel.STL"
-          mass="0.08" >
+          mass="0.08">
           <origin
                xyz="3.8886E-14 3.645E-14 0.38665"
@@ -81,7 +84,7 @@
      <!-- <IMU> -->
      <!-- <Lidar> -->
-     <xacro:lidar_link
+     <xacro:lidar_m
           filename="package://description/meshes/lidar_link.STL"
-          mass = "0.25" >
+          mass="0.25" >
           <origin
                xyz="0.00012979 -6.6734E-06 -0.0079009"
@@ -96,5 +99,5 @@
                izz="1.7083E-05"
           />
-     </xacro:lidar_link>
+     </xacro:lidar_m>
      <xacro:lidar_joint>
           <origin
@@ -105,8 +108,7 @@
      <!-- <Lidar> -->
      <!-- <Aruco> -->
-     <xacro:aruco>
-          <box size="0.10 0.10 0.02" />
+     <xacro:aruco_m>
           <origin xyz="-0.09 0 0.26" rpy="0 0 0" />
-     </xacro:aruco>
+     </xacro:aruco_m>
      <!-- <Aruco> -->
 </robot>

File: src/ros2/description/urdf/robot.urdf.xacro (robot description, xacro)
@@ -1,3 +1,3 @@
-<?xml version="1.0"?>
+<?xml version="1.0" encoding="utf-8"?>
 <robot xmlns:xacro="http://www.ros.org/wiki/xacro"  name="Maket">
     <xacro:include filename="descriptions.xacro"/>

File: src/ros2/description/urdf/sensors.xacro (robot description, xacro)
@@ -1,7 +1,7 @@
-<?xml version="1.0"?>
+<?xml version="1.0" encoding="utf-8"?>
 <robot xmlns:xacro="http://ros.org/wiki/xacro">
-  <material name = "lidar">
+  <material name="lidar_material">
     <color
-      rgba = "0 1 0 1" />
+      rgba="0 1 0 1" />
   </material>
   <xacro:macro name="imu">
@@ -13,5 +13,5 @@
     </joint>
   </xacro:macro>
-  <xacro:macro name="lidar_link" params="filename mass *origin *inertia">
+  <xacro:macro name="lidar_m" params="filename mass *origin *inertia">
     <link name="lidar_link">
       <visual>
@@ -23,5 +23,5 @@
           <mesh filename="${filename}" />
         </geometry>
-        <material name = "lidar"/>
+        <material name="lidar_material"/>
       </visual>
       <collision>
@@ -41,5 +41,5 @@
     </link>
   </xacro:macro>
-  <xacro:macro name = "lidar_joint" params = "*origin">
+  <xacro:macro name="lidar_joint" params="*origin">
     <joint name="lidar_to_base" type="fixed">
       <parent link="base_link"/>

File: src/ros2/description/urdf/structure.xacro (robot description, xacro)
@@ -2,19 +2,15 @@
 <robot xmlns:xacro="http://www.ros.org/wiki/xacro" >
     <!-- Specify some colours -->
-    <material name="base_link">
+    <material name="base_material">
         <color
           rgba="1 0 0 1" />
     </material>
-    <material name="right_wheel">
-        <color
-          rgba="0 0 1 1" />
-    </material>
-    <material name="left_wheel">
+    <material name="wheel_material">
         <color
           rgba="0 0 1 1" />
     </material>
     <!-- Macros for base_link-->
-    <xacro:macro name="base_link" params="name mass filename *origin *inertia">
-        <link name = "${name}">
+    <xacro:macro name="base_m" params="name mass filename *origin *inertia">
+        <link name="${name}">
             <visual>
                 <origin
@@ -25,5 +21,5 @@
                     <mesh filename="${filename}" />
                 </geometry>
-                <material name="base_link" />
+                <material name="base_material" />
             </visual>
             <collision>
@@ -33,17 +29,17 @@
                 />
                 <geometry>
-                    <mesh filename = "${filename}" />
+                    <mesh filename="${filename}" />
                 </geometry>
             </collision>
             <inertial>
-                <xacro:insert_block name = "origin" />
-                <mass value = "${mass}" />
-                <xacro:insert_block name = "inertia" />
+                <xacro:insert_block name="origin" />
+                <mass value="${mass}" />
+                <xacro:insert_block name="inertia" />
             </inertial>
         </link>
     </xacro:macro>
     <!-- Macros for wheels links & joints-->
-    <xacro:macro name = "wheel_link" params="name_link filename mass *origin *inertia" >
-          <link name = "${name_link}">
+    <xacro:macro name="wheel_link" params="name_link filename mass *origin *inertia" >
+          <link name="${name_link}">
                <visual>
                     <origin
@@ -52,7 +48,7 @@
                     />
                     <geometry>
-                         <mesh filename = "${filename}" />
+                         <mesh filename="${filename}" />
                     </geometry>
-                    <material name = "${name_link}" />
+                    <material name="wheel_material" />
                </visual>
                <collision>
@@ -62,19 +58,19 @@
                     />
                     <geometry>
-                         <mesh filename = "${filename}" />
+                         <mesh filename="${filename}" />
                     </geometry>
                </collision>
                <inertial>
                     <xacro:insert_block name="origin" />
-                    <mass = "${mass}" />
+                    <mass value="${mass}" />
                     <xacro:insert_block name="inertia" />
                </inertial>
           </link>
      </xacro:macro>
-     <xacro:macro name = "wheel_joint" params = "name name_link *origin">
-          <joint name = "${name}" type = "continuous">
+     <xacro:macro name="wheel_joint" params="name name_link *origin">
+          <joint name="${name}" type="continuous">
                <xacro:insert_block name="origin" />
-               <parent link = "base_link" />
-               <child link = "${name_link}" />
+               <parent link="base_link" />
+               <child link="${name_link}" />
                <axis xyz="0 0 1" />
                <limit
@@ -89,17 +85,17 @@
      </xacro:macro>
     <!-- Macros for aruco link-->
-    <xacro:macro name = "aruco" params ="*box *origin">
+    <xacro:macro name="aruco_str" params ="material *origin">
         <link name="aruco">
             <visual>
                 <origin xyz="0 0 0" rpy="0 0 0" />
                 <geometry>
-                    <xacro:insert_block name="box" />
+                    <box size="0.10 0.10 0.02" />
                 </geometry>
-                <material name="right_wheel" />
+                <material name="wheel_material" />
             </visual>
             <collision>
                 <origin xyz="0 0 0" rpy="0 0 0" />
                 <geometry>
-                        <xacro:insert_block name="box" />
+                        <box size="0.10 0.10 0.02" />
                 </geometry>
             </collision>

Commit message: URDF for model v2.0 + meshes

File: src/ros2/description/urdf/descriptions.xacro (robot description, xacro)
@@ -14,14 +14,14 @@
           filename="package://description/meshes/base_link.STL">
           <origin
-               xyz="0.055795 0.00111 0.11345"
+               xyz="0.024636 0.00068431 0.10638"
                rpy="0 0 0"
           />
           <inertia
-               ixx="0.01219"
-               ixy="0.00012117"
-               ixz="0.00018358"
-               iyy="0.0027513"
-               iyz="-0.00011927"
-               izz="0.012455"
+               ixx="0.018097"
+               ixy="8.6144E-05"
+               ixz="6.7135E-05"
+               iyy="0.0070038"
+               iyz="-9.0076E-05"
+               izz="0.01647"
           />
      </xacro:base_m>
@@ -32,13 +32,13 @@
           mass="0.08">
           <origin
-               xyz="8.3267E-17 0 0.013353"
+               xyz="0 -8.6254E-14 0.013353"
                rpy="0 0 0"
           />
           <inertia
                ixx="3.6651E-05"
-               ixy="1.1089E-20"
-               ixz="1.0295E-19"
+               ixy="9.6988E-21"
+               ixz="-7.7529E-22"
                iyy="3.6651E-05"
-               iyz="2.2675E-21"
+               iyz="-1.1318E-16"
                izz="5.4175E-05"
           />
@@ -48,5 +48,5 @@
           name_link="right_wheel">
           <origin
-               xyz="0.059148 -0.2 0.021"
+               xyz="0.059075 -0.2 0.021"
                rpy="-1.5708 0 0"
           />
@@ -59,13 +59,13 @@
           mass="0.08">
           <origin
-               xyz="3.8886E-14 3.645E-14 0.38665"
+               xyz="6.8279E-15 -1.2143E-15 -0.013353"
                rpy="0 0 0"
           />
           <inertia
                ixx="3.6651E-05"
-               ixy="-1.2633E-21"
-               ixz="-9.0385E-18"
+               ixy="-1.3538E-21"
+               ixz="-8.9321E-18"
                iyy="3.6651E-05"
-               iyz="7.177E-19"
+               iyz="1.5999E-18"
                izz="5.4175E-05"
           />
@@ -75,5 +75,5 @@
           name_link="left_wheel">
           <origin
-               xyz="0.059148 -0.2 0.021"
+               xyz="0.059075 0.2 0.021"
                rpy="-1.5708 0 0"
           />
@@ -84,31 +84,47 @@
      <!-- <IMU> -->
      <!-- <Lidar> -->
-     <xacro:lidar_m
+     <xacro:lidar_link_m
           filename="package://description/meshes/lidar_link.STL"
           mass="0.25" >
           <origin
-               xyz="0.00012979 -6.6734E-06 -0.0079009"
+               xyz="0.0001471 4.608E-08 -0.015129"
                rpy="0 0 0"
           />
           <inertia
                ixx="9.5253E-06"
-               ixy="6.45E-11"
-               ixz="4.1315E-08"
-               iyy="9.4166E-06"
-               iyz="6.3454E-09"
+               ixy="4.0169E-10"
+               ixz="2.4656E-08"
+               iyy="9.4165E-06"
+               iyz="-9.4826E-12"
                izz="1.7083E-05"
           />
-     </xacro:lidar_m>
-     <xacro:lidar_joint>
+     </xacro:lidar_link_m>
+     <xacro:lidar_joint_m>
           <origin
-               xyz="0.005563 0.002859 0.30015"
+               xyz="-0.0032264 0 0.31758"
                rpy="0 0 0"
           />
-     </xacro:lidar_joint>
+     </xacro:lidar_joint_m>
      <!-- <Lidar> -->
      <!-- <Aruco> -->
-     <xacro:aruco_m>
-          <origin xyz="-0.09 0 0.26" rpy="0 0 0" />
-     </xacro:aruco_m>
+     <xacro:aruco_link_m
+          filename="package://description/meshes/aruco_link.STL"
+          mass="0.2">
+          <origin
+               xyz="-0.0092221 -1.2598E-17 -0.044216"
+               rpy="0 0 0" />
+          <inertia
+               ixx="0.00036111"
+               ixy="-1.6666E-21"
+               ixz="-6.4905E-05"
+               iyy="0.0003976"
+               iyz="1.3655E-19"
+               izz="0.00040158" />
+     </xacro:aruco_link_m>
+     <xacro:aruco_joint_m>
+          <origin
+          xyz="-0.0032264 0 0.411"
+          rpy="0 0 0" />
+     </xacro:aruco_joint_m>
      <!-- <Aruco> -->
 </robot>

File: src/ros2/description/urdf/sensors.xacro (robot description, xacro)
@@ -3,5 +3,5 @@
   <material name="lidar_material">
     <color
-      rgba="0 1 0 1" />
+      rgba="1 1 1 1" />
   </material>
   <xacro:macro name="imu">
@@ -13,5 +13,5 @@
     </joint>
   </xacro:macro>
-  <xacro:macro name="lidar_m" params="filename mass *origin *inertia">
+  <xacro:macro name="lidar_link_m" params="filename mass *origin *inertia">
     <link name="lidar_link">
       <visual>
@@ -41,18 +41,9 @@
     </link>
   </xacro:macro>
-  <xacro:macro name="lidar_joint" params="*origin">
+  <xacro:macro name="lidar_joint_m" params="*origin">
     <joint name="lidar_to_base" type="fixed">
       <parent link="base_link"/>
       <child link="lidar_link"/>
       <xacro:insert_block name="origin" />
-      <axis xyz="0 0 0" />
-      <limit
-        effort="0"
-        velocity="0"
-      />
-      <dynamics
-        damping="0"
-        friction="0"
-      />
     </joint>
   </xacro:macro>

File: src/ros2/description/urdf/structure.xacro (robot description, xacro)
@@ -9,4 +9,8 @@
         <color
           rgba="0 0 1 1" />
+    </material>
+    <material name="aruco_material">
+        <color
+            rgba="0 1 0 1" />
     </material>
     <!-- Macros for base_link-->
@@ -85,24 +89,32 @@
      </xacro:macro>
     <!-- Macros for aruco link-->
-    <xacro:macro name="aruco_str" params ="material *origin">
-        <link name="aruco">
+    <xacro:macro name="aruco_link_m" params ="filename mass *origin *inertia">
+        <link name="aruco_link">
             <visual>
                 <origin xyz="0 0 0" rpy="0 0 0" />
                 <geometry>
-                    <box size="0.10 0.10 0.02" />
+                    <mesh filename="${filename}" />
                 </geometry>
-                <material name="wheel_material" />
+                <material name="aruco_material" />
             </visual>
             <collision>
                 <origin xyz="0 0 0" rpy="0 0 0" />
                 <geometry>
-                        <box size="0.10 0.10 0.02" />
+                    <mesh filename="${filename}" />
                 </geometry>
             </collision>
+            <inertial>
+                <xacro:insert_block name="origin" />
+                <mass value="${mass}" />
+                <xacro:insert_block name="inertia" />
+            </inertial>
         </link>
-        <joint name="aruco" type="fixed">
-          <parent link="base_link" />
-          <child link="aruco" />
-          <xacro:insert_block name="origin" />
+    </xacro:macro>
+    <xacro:macro name="aruco_joint_m" params="*origin">
+        <joint name="aruco_to_base" type="fixed">
+            <xacro:insert_block name="origin" />
+            <parent link="base_link" />
+            <child link="aruco_link" />
+            <axis xyz="0 0 0" />
         </joint>
     </xacro:macro>

Commit message: fix: Some refatoring

File: src/ros2/description/urdf/descriptions.xacro (robot description, xacro)
@@ -2,5 +2,5 @@
 <robot xmlns:xacro="http://www.ros.org/wiki/xacro" name="Maket">
      <xacro:include filename="inertials.xacro" />
-     <xacro:include filename="sensors.urdf.xacro" />
+     <xacro:include filename="sensors.xacro" />
      <link name="base_footprint" />
      <joint name="base_to_footprint" type="fixed">
@@ -127,5 +127,5 @@
      <xacro:imu />
      <xacro:laser>
-          <origin xyz="0 0 0.33" rpy="0 0 0" />
+          <origin xyz="0 0 0.33" rpy="0 0 3.14" />
      </xacro:laser>
      <link name="aruco">

File: src/ros2/description/urdf/sensors.xacro (robot description, xacro)
@@ -6,5 +6,5 @@
       <parent link="base_link"/>
       <child link="imu_link"/>
-      <origin xyz="0 0 0" rpy="3.14 0 0"/>
+      <origin xyz="0 0 0" rpy="0 0 0"/>
     </joint>
   </xacro:macro>
