Commit message: Prepare to merge

File: src/ros2/description/urdf/descriptions.xacro (robot description, xacro)
@@ -9,121 +9,52 @@
           <origin xyz="0 0 0" rpy="0 0 0" />
      </joint>
-     <xacro:base_m
-          name="base_link"
-          mass="5"
-          filename="package://description/meshes/base_link.STL">
-          <origin
-               xyz="0.024636 0.00068431 0.10638"
-               rpy="0 0 0"
-          />
-          <inertia
-               ixx="0.018097"
-               ixy="8.6144E-05"
-               ixz="6.7135E-05"
-               iyy="0.0070038"
-               iyz="-9.0076E-05"
-               izz="0.01647"
-          />
+     <xacro:base_m name="base_link" mass="5" filename="package://description/meshes/base_link.STL">
+          <origin xyz="0.024636 0.00068431 0.10638" rpy="0 0 0" />
+          <inertia ixx="0.018097" ixy="8.6144E-05" ixz="6.7135E-05" iyy="0.0070038"
+               iyz="-9.0076E-05" izz="0.01647" />
      </xacro:base_m>
      <!-- <Right_Wheel> -->
-     <xacro:wheel_link
-          name_link="right_wheel"
-          filename="package://description/meshes/right_wheel.STL"
-          mass="0.08">
-          <origin
-               xyz="0 -8.6254E-14 0.013353"
-               rpy="0 0 0"
-          />
-          <inertia
-               ixx="3.6651E-05"
-               ixy="9.6988E-21"
-               ixz="-7.7529E-22"
-               iyy="3.6651E-05"
-               iyz="-1.1318E-16"
-               izz="5.4175E-05"
-          />
+     <xacro:wheel_link name_link="right_wheel"
+          filename="package://description/meshes/right_wheel.STL" mass="0.08">
+          <origin xyz="0 -8.6254E-14 0.013353" rpy="0 0 0" />
+          <inertia ixx="3.6651E-05" ixy="9.6988E-21" ixz="-7.7529E-22" iyy="3.6651E-05"
+               iyz="-1.1318E-16" izz="5.4175E-05" />
      </xacro:wheel_link>
-     <xacro:wheel_joint
-          name="rightwheel"
-          name_link="right_wheel">
-          <origin
-               xyz="0.059075 -0.2 0.021"
-               rpy="-1.5708 0 0"
-          />
+     <xacro:wheel_joint name="rightwheel" name_link="right_wheel">
+          <origin xyz="0.059075 -0.2 0.021" rpy="-1.5708 0 0" />
      </xacro:wheel_joint>
      <!-- </Right_Wheel> -->
      <!-- <Left_Wheel> -->
-     <xacro:wheel_link
-          name_link="left_wheel"
-          filename="package://description/meshes/left_wheel.STL"
+     <xacro:wheel_link name_link="left_wheel" filename="package://description/meshes/left_wheel.STL"
           mass="0.08">
-          <origin
-               xyz="6.8279E-15 -1.2143E-15 -0.013353"
-               rpy="0 0 0"
-          />
-          <inertia
-               ixx="3.6651E-05"
-               ixy="-1.3538E-21"
-               ixz="-8.9321E-18"
-               iyy="3.6651E-05"
-               iyz="1.5999E-18"
-               izz="5.4175E-05"
-          />
+          <origin xyz="6.8279E-15 -1.2143E-15 -0.013353" rpy="0 0 0" />
+          <inertia ixx="3.6651E-05" ixy="-1.3538E-21" ixz="-8.9321E-18" iyy="3.6651E-05"
+               iyz="1.5999E-18" izz="5.4175E-05" />
      </xacro:wheel_link>
-     <xacro:wheel_joint
-          name="leftwheel"
-          name_link="left_wheel">
-          <origin
-               xyz="0.059075 0.2 0.021"
-               rpy="-1.5708 0 0"
-          />
+     <xacro:wheel_joint name="leftwheel" name_link="left_wheel">
+          <origin xyz="0.059075 0.2 0.021" rpy="-1.5708 0 0" />
      </xacro:wheel_joint>
      <!-- <Left_Wheel> -->
      <!-- <IMU> -->
-     <xacro:imu/>
+     <xacro:imu />
      <!-- <IMU> -->
      <!-- <Lidar> -->
-     <xacro:lidar_link_m
-          filename="package://description/meshes/lidar_link.STL"
-          mass="0.25" >
-          <origin
-               xyz="0.0001471 4.608E-08 -0.015129"
-               rpy="0 0 0"
-          />
-          <inertia
-               ixx="9.5253E-06"
-               ixy="4.0169E-10"
-               ixz="2.4656E-08"
-               iyy="9.4165E-06"
-               iyz="-9.4826E-12"
-               izz="1.7083E-05"
-          />
+     <xacro:lidar_link_m filename="package://description/meshes/lidar_link.STL" mass="0.25">
+          <origin xyz="0.0001471 4.608E-08 -0.015129" rpy="0 0 0" />
+          <inertia ixx="9.5253E-06" ixy="4.0169E-10" ixz="2.4656E-08" iyy="9.4165E-06"
+               iyz="-9.4826E-12" izz="1.7083E-05" />
      </xacro:lidar_link_m>
      <xacro:lidar_joint_m>
-          <origin
-               xyz="-0.0032264 0 0.31758"
-               rpy="0 0 0"
-          />
+          <origin xyz="-0.0032264 0 0.31758" rpy="0 0 0" />
      </xacro:lidar_joint_m>
      <!-- <Lidar> -->
      <!-- <Aruco> -->
-     <xacro:aruco_link_m
-          filename="package://description/meshes/aruco_link.STL"
-          mass="0.2">
-          <origin
-               xyz="-0.0092221 -1.2598E-17 -0.044216"
-               rpy="0 0 0" />
-          <inertia
-               ixx="0.00036111"
-               ixy="-1.6666E-21"
-               ixz="-6.4905E-05"
-               iyy="0.0003976"
-               iyz="1.3655E-19"
-               izz="0.00040158" />
+     <xacro:aruco_link_m filename="package://description/meshes/aruco_link.STL" mass="0.2">
+          <origin xyz="-0.0092221 -1.2598E-17 -0.044216" rpy="0 0 0" />
+          <inertia ixx="0.00036111" ixy="-1.6666E-21" ixz="-6.4905E-05" iyy="0.0003976"
+               iyz="1.3655E-19" izz="0.00040158" />
      </xacro:aruco_link_m>
      <xacro:aruco_joint_m>
-          <origin
-          xyz="-0.0032264 0 0.411"
-          rpy="0 0 0" />
+          <origin xyz="-0.0032264 0 0.411" rpy="0 0 0" />
      </xacro:aruco_joint_m>
      <!-- <Aruco> -->

File: src/ros2/description/urdf/robot.urdf.xacro (robot description, xacro)
@@ -1,4 +1,4 @@
 <?xml version="1.0" encoding="utf-8"?>
-<robot xmlns:xacro="http://www.ros.org/wiki/xacro"  name="Maket">
-    <xacro:include filename="descriptions.xacro"/>
+<robot xmlns:xacro="http://www.ros.org/wiki/xacro" name="Maket">
+    <xacro:include filename="descriptions.xacro" />
 </robot>

File: src/ros2/description/urdf/sensors.xacro (robot description, xacro)
@@ -6,9 +6,9 @@
   </material>
   <xacro:macro name="imu">
-    <link name="imu_link"/>
+    <link name="imu_link" />
     <joint name="imu_to_base_link" type="fixed">
-      <parent link="base_link"/>
-      <child link="imu_link"/>
-      <origin xyz="0 0 0" rpy="3.14 0 0"/>
+      <parent link="base_link" />
+      <child link="imu_link" />
+      <origin xyz="0 0 0" rpy="3.14 0 0" />
     </joint>
   </xacro:macro>
@@ -23,5 +23,5 @@
           <mesh filename="${filename}" />
         </geometry>
-        <material name="lidar_material"/>
+        <material name="lidar_material" />
       </visual>
       <collision>
@@ -36,5 +36,5 @@
       <inertial>
         <xacro:insert_block name="origin" />
-        <mass value="${mass}"/>
+        <mass value="${mass}" />
         <xacro:insert_block name="inertia" />
       </inertial>
@@ -43,6 +43,6 @@
   <xacro:macro name="lidar_joint_m" params="*origin">
     <joint name="lidar_to_base" type="fixed">
-      <parent link="base_link"/>
-      <child link="lidar_link"/>
+      <parent link="base_link" />
+      <child link="lidar_link" />
       <xacro:insert_block name="origin" />
     </joint>

File: src/ros2/description/urdf/structure.xacro (robot description, xacro)
@@ -1,12 +1,12 @@
 <?xml version="1.0" encoding="utf-8"?>
-<robot xmlns:xacro="http://www.ros.org/wiki/xacro" >
+<robot xmlns:xacro="http://www.ros.org/wiki/xacro">
     <!-- Specify some colours -->
     <material name="base_material">
         <color
-          rgba="1 0 0 1" />
+            rgba="1 0 0 1" />
     </material>
     <material name="wheel_material">
         <color
-          rgba="0 0 1 1" />
+            rgba="0 0 1 1" />
     </material>
     <material name="aruco_material">
@@ -44,50 +44,50 @@
     </xacro:macro>
     <!-- Macros for wheels links & joints-->
-    <xacro:macro name="wheel_link" params="name_link filename mass *origin *inertia" >
-          <link name="${name_link}">
-               <visual>
-                    <origin
-                        xyz="0 0 0"
-                        rpy="0 0 0"
-                    />
-                    <geometry>
-                         <mesh filename="${filename}" />
-                    </geometry>
-                    <material name="wheel_material" />
-               </visual>
-               <collision>
-                    <origin
-                        xyz="0 0 0"
-                        rpy="0 0 0"
-                    />
-                    <geometry>
-                         <mesh filename="${filename}" />
-                    </geometry>
-               </collision>
-               <inertial>
-                    <xacro:insert_block name="origin" />
-                    <mass value="${mass}" />
-                    <xacro:insert_block name="inertia" />
-               </inertial>
-          </link>
-     </xacro:macro>
-     <xacro:macro name="wheel_joint" params="name name_link *origin">
-          <joint name="${name}" type="continuous">
-               <xacro:insert_block name="origin" />
-               <parent link="base_link" />
-               <child link="${name_link}" />
-               <axis xyz="0 0 1" />
-               <limit
-                    effort="0"
-                    velocity="10"
-               />
-               <dynamics
-                    damping="0"
-                    friction="0"
-               />
-          </joint>
-     </xacro:macro>
+    <xacro:macro name="wheel_link" params="name_link filename mass *origin *inertia">
+        <link name="${name_link}">
+            <visual>
+                <origin
+                    xyz="0 0 0"
+                    rpy="0 0 0"
+                />
+                <geometry>
+                    <mesh filename="${filename}" />
+                </geometry>
+                <material name="wheel_material" />
+            </visual>
+            <collision>
+                <origin
+                    xyz="0 0 0"
+                    rpy="0 0 0"
+                />
+                <geometry>
+                    <mesh filename="${filename}" />
+                </geometry>
+            </collision>
+            <inertial>
+                <xacro:insert_block name="origin" />
+                <mass value="${mass}" />
+                <xacro:insert_block name="inertia" />
+            </inertial>
+        </link>
+    </xacro:macro>
+    <xacro:macro name="wheel_joint" params="name name_link *origin">
+        <joint name="${name}" type="continuous">
+            <xacro:insert_block name="origin" />
+            <parent link="base_link" />
+            <child link="${name_link}" />
+            <axis xyz="0 0 1" />
+            <limit
+                effort="0"
+                velocity="10"
+            />
+            <dynamics
+                damping="0"
+                friction="0"
+            />
+        </joint>
+    </xacro:macro>
     <!-- Macros for aruco link-->
-    <xacro:macro name="aruco_link_m" params ="filename mass *origin *inertia">
+    <xacro:macro name="aruco_link_m" params="filename mass *origin *inertia">
         <link name="aruco_link">
             <visual>

Commit message: Stable version with model 2.0

File: src/ros2/description/urdf/descriptions.xacro (robot description, xacro)
@@ -40,12 +40,12 @@
      <!-- <IMU> -->
      <!-- <Lidar> -->
-     <xacro:lidar_link_m filename="package://description/meshes/lidar_link.STL" mass="0.25">
-          <origin xyz="0.0001471 4.608E-08 -0.015129" rpy="0 0 0" />
-          <inertia ixx="9.5253E-06" ixy="4.0169E-10" ixz="2.4656E-08" iyy="9.4165E-06"
-               iyz="-9.4826E-12" izz="1.7083E-05" />
-     </xacro:lidar_link_m>
-     <xacro:lidar_joint_m>
+     <xacro:laser >
           <origin xyz="-0.0032264 0 0.31758" rpy="0 0 0" />
-     </xacro:lidar_joint_m>
+          <!-- <inertia ixx="9.5253E-06" ixy="4.0169E-10" ixz="2.4656E-08" iyy="9.4165E-06"
+               iyz="-9.4826E-12" izz="1.7083E-05" /> -->
+     </xacro:laser>
+     <!-- <xacro:lidar_to_base_link>
+          <origin xyz="-0.0032264 0 0.31758" rpy="0 0 0" />
+     </xacro:lidar_to_base_link> -->
      <!-- <Lidar> -->
      <!-- <Aruco> -->

Commit message: maket v2.2 to urdf

File: src/ros2/description/urdf/descriptions.xacro (robot description, xacro)
@@ -14,15 +14,14 @@
           filename="package://description/meshes/base_link.STL">
           <origin
-               xyz="0.024636 0.00068431 0.10638"
+               xyz="0.016054 -0.0031971 0.10841"
                rpy="0 0 0"
           />
           <inertia
-               ixx="0.018097"
-               ixy="8.6144E-05"
-               ixz="6.7135E-05"
-               iyy="0.0070038"
-               iyz="-9.0076E-05"
-               izz="0.01647"
-          />
+          ixx="0.019114"
+          ixy="0.00015199"
+          ixz="6.8537E-05"
+          iyy="0.0061796"
+          iyz="-9.0111E-05"
+          izz="0.019044" />
      </xacro:base_m>
      <!-- <Right_Wheel> -->
@@ -32,5 +31,5 @@
           mass="0.08">
           <origin
-               xyz="0 -8.6254E-14 0.013353"
+               xyz="-6.245E-17 -2.8449E-16 0.013347"
                rpy="0 0 0"
           />
@@ -48,5 +47,5 @@
           name_link="right_wheel">
           <origin
-               xyz="0.059075 -0.2 0.021"
+               xyz="0.058997 -0.2 0.021"
                rpy="-1.5708 0 0"
           />
@@ -59,13 +58,13 @@
           mass="0.08">
           <origin
-               xyz="6.8279E-15 -1.2143E-15 -0.013353"
+               xyz="4.5103E-17 2.0817E-17 -0.013347"
                rpy="0 0 0"
           />
           <inertia
-               ixx="3.6651E-05"
-               ixy="-1.3538E-21"
-               ixz="-8.9321E-18"
-               iyy="3.6651E-05"
-               iyz="1.5999E-18"
+               ixx="3.6634E-05"
+               ixy="1.2292E-20"
+               ixz="-5.2555E-20"
+               iyy="3.6634E-05"
+               iyz="-3.185E-20"
                izz="5.4175E-05"
           />
@@ -75,5 +74,5 @@
           name_link="left_wheel">
           <origin
-               xyz="0.059075 0.2 0.021"
+               xyz="0.058997 0.2 0.021"
                rpy="-1.5708 0 0"
           />
@@ -84,6 +83,8 @@
      <!-- <IMU> -->
      <!-- <Lidar> -->
-     <xacro:lidar_link_m
-          filename="package://description/meshes/lidar_link.STL"
+     <xacro:lazer
+          xyz="0 0 0.308"
+          length="0.041"
+          radius="0.040"
           mass="0.25" >
           <origin
@@ -91,38 +92,24 @@
                rpy="0 0 0"
           />
-          <inertia
-               ixx="9.5253E-06"
-               ixy="4.0169E-10"
-               ixz="2.4656E-08"
-               iyy="9.4165E-06"
-               iyz="-9.4826E-12"
-               izz="1.7083E-05"
-          />
-     </xacro:lidar_link_m>
-     <xacro:lidar_joint_m>
-          <origin
-               xyz="-0.0032264 0 0.31758"
-               rpy="0 0 0"
-          />
-     </xacro:lidar_joint_m>
+     </xacro:lazer>
      <!-- <Lidar> -->
      <!-- <Aruco> -->
      <xacro:aruco_link_m
           filename="package://description/meshes/aruco_link.STL"
-          mass="0.2">
+          mass="0.4">
           <origin
-               xyz="-0.0092221 -1.2598E-17 -0.044216"
+               xyz="-0.0077972 5.7506E-10 -0.038759"
                rpy="0 0 0" />
           <inertia
-               ixx="0.00036111"
-               ixy="-1.6666E-21"
-               ixz="-6.4905E-05"
-               iyy="0.0003976"
-               iyz="1.3655E-19"
-               izz="0.00040158" />
+               ixx="0.00060095"
+               ixy="1.109E-09"
+               ixz="-0.00011373"
+               iyy="0.00065092"
+               iyz="-2.1703E-12"
+               izz="0.00071676" />
      </xacro:aruco_link_m>
      <xacro:aruco_joint_m>
           <origin
-          xyz="-0.0032264 0 0.411"
+          xyz="-0.003304 0 0.431"
           rpy="0 0 0" />
      </xacro:aruco_joint_m>

File: src/ros2/description/urdf/sensors.xacro (robot description, xacro)
@@ -13,13 +13,13 @@
     </joint>
   </xacro:macro>
-  <xacro:macro name="lidar_link_m" params="filename mass *origin *inertia">
+  <xacro:macro name="lazer" params="xyz,length,radius,mass,*origin">
     <link name="lidar_link">
       <visual>
         <origin
-          xyz="0 0 0"
+          xyz="${xyz}"
           rpy="0 0 0"
         />
         <geometry>
-          <mesh filename="${filename}" />
+          <cylinder length="${length}" radius="${radius}" />
         </geometry>
         <material name="lidar_material"/>
@@ -27,9 +27,9 @@
       <collision>
         <origin
-          xyz="0 0 0"
+          xyz="${xyz}"
           rpy="0 0 0"
         />
         <geometry>
-          <mesh filename="${filename}" />
+          <cylinder length="${length}" radius="${radius}" />
         </geometry>
       </collision>
@@ -37,14 +37,9 @@
         <xacro:insert_block name="origin" />
         <mass value="${mass}"/>
-        <xacro:insert_block name="inertia" />
+        <inertia ixx="${(1/12) * mass * (3*radius*radius + length*length)}" ixy="0.0" ixz="0.0"
+                    iyy="${(1/12) * mass * (3*radius*radius + length*length)}" iyz="0.0"
+                    izz="${(1/2) * mass * (radius*radius)}" />
       </inertial>
     </link>
   </xacro:macro>
-  <xacro:macro name="lidar_joint_m" params="*origin">
-    <joint name="lidar_to_base" type="fixed">
-      <parent link="base_link"/>
-      <child link="lidar_link"/>
-      <xacro:insert_block name="origin" />
-    </joint>
-  </xacro:macro>
 </robot>

Commit message: lidar_lockalization working prototype

File: src/ros2/description/urdf/descriptions.xacro (robot description, xacro)
@@ -41,5 +41,5 @@
      <!-- <Lidar> -->
      <xacro:laser >
-          <origin xyz="-0.0032264 0 0.31758" rpy="0 0 0" />
+          <origin xyz="-0.0032264 0 0.31758" rpy="0 0 3.14" />
           <!-- <inertia ixx="9.5253E-06" ixy="4.0169E-10" ixz="2.4656E-08" iyy="9.4165E-06"
                iyz="-9.4826E-12" izz="1.7083E-05" /> -->

Commit message: Fix after merge. All works clean!

File: src/ros2/description/urdf/descriptions.xacro (robot description, xacro)
@@ -83,16 +83,13 @@
      <xacro:lazer
           xyz="0 0 0.308"
+          rpy = "0 0 180"
           length="0.041"
           radius="0.040"
           mass="0.25" >
-          <origin
-               xyz="0.0001471 4.608E-08 -0.015129"
-               rpy="0 0 0"
-          />
      </xacro:lazer>
      <!-- <Lidar> -->
      <!-- <Aruco> -->
      <xacro:aruco_link_m
-          filename="package://description/meshes/aruco_link.STL"
+          filename="package://description/meshes/aruco.STL"
           mass="0.4">
           <origin

File: src/ros2/description/urdf/sensors.xacro (robot description, xacro)
@@ -13,33 +13,35 @@
     </joint>
   </xacro:macro>
-  <xacro:macro name="lazer" params="xyz,length,radius,mass,*origin">
-    <link name="lidar_link">
-      <visual>
-        <origin
-          xyz="${xyz}"
-          rpy="0 0 0"
-        />
-        <geometry>
-          <cylinder length="${length}" radius="${radius}" />
-        </geometry>
-        <material name="lazer_material"/>
-      </visual>
-      <collision>
-        <origin
-          xyz="${xyz}"
-          rpy="0 0 0"
-        />
-        <geometry>
-          <cylinder length="${length}" radius="${radius}" />
-        </geometry>
-      </collision>
-      <inertial>
-        <xacro:insert_block name="origin" />
-        <mass value="${mass}"/>
-        <inertia ixx="${(1/12) * mass * (3*radius*radius + length*length)}" ixy="0.0" ixz="0.0"
-                    iyy="${(1/12) * mass * (3*radius*radius + length*length)}" iyz="0.0"
-                    izz="${(1/2) * mass * (radius*radius)}" />
-      </inertial>
-    </link>
-  </xacro:macro>
+  <xacro:macro name="lazer" params="xyz rpy length radius mass">
+  <link name="lidar_link">
+    <visual>
+      <origin xyz="0 0 0" rpy="0 0 0"/>
+      <geometry>
+        <cylinder length="${length}" radius="${radius}"/>
+      </geometry>
+      <material name="lazer_material"/>
+    </visual>
+    <collision>
+      <origin xyz="${xyz}" rpy="${rpy}"/>
+      <geometry>
+        <cylinder length="${length}" radius="${radius}"/>
+      </geometry>
+    </collision>
+    <inertial>
+      <!-- Provide a default origin for inertial properties -->
+      <origin xyz="${xyz}" rpy="${rpy}"/>
+      <mass value="${mass}"/>
+      <inertia ixx="${(1/12) * mass * (3*(radius*radius) + (length*length))}"
+               ixy="0.0" ixz="0.0"
+               iyy="${(1/12) * mass * (3*(radius*radius) + (length*length))}"
+               iyz="0.0"
+               izz="${(1/2) * mass * (radius*radius)}"/>
+    </inertial>
+  </link>
+  <joint name="lidar_to_base_link" type="fixed">
+      <parent link="base_link"/>
+      <child link="lidar_link"/>
+      <origin xyz="${xyz}" rpy="${rpy}"/>
+  </joint>
+</xacro:macro>
 </robot>
