Commit message: STL URDF fix

File: src/ros2/description/urdf/sensors.xacro (robot description, xacro)
@@ -1,4 +1,8 @@
-<?xml version="1.0"?>
+<?xml version="1.0" encoding="utf-8"?>
 <robot xmlns:xacro="http://ros.org/wiki/xacro">
+   <material name="lazer_material">
+      <color
+        rgba="1 1 1 1" />
+      </material>
   <xacro:macro name="imu">
     <link name="imu_link"/>
@@ -19,7 +23,5 @@
           <cylinder length="${length}" radius="${radius}" />
         </geometry>
-        <material name="green">
-            <color rgba="0.003 0.639 0.223 1.0"/>
-        </material>
+        <material name="lazer_material"/>
       </visual>
       <collision>

Commit message: set up camera+lidar localization.
Start setting up navigation.yaml

File: src/ros2/description/urdf/sensors.xacro (robot description, xacro)
@@ -10,5 +10,5 @@
       <parent link="base_link"/>
       <child link="imu_link"/>
-      <origin xyz="0 0 0" rpy="0 0 0"/>
+      <origin xyz="0.065 0 0" rpy="0 0 0"/>
     </joint>
   </xacro:macro>

Commit message: new imu implementation

File: src/ros2/description/urdf/sensors.xacro (robot description, xacro)
@@ -6,9 +6,9 @@
       </material>
   <xacro:macro name="imu">
-    <link name="imu_link"/>
+    <link name="base_imu_link"/>
     <joint name="imu_to_base_link" type="fixed">
       <parent link="base_link"/>
-      <child link="imu_link"/>
-      <origin xyz="0.065 0 0" rpy="0 0 0"/>
+      <child link="base_imu_link"/>
+      <origin xyz="0.065 0 0" rpy="0 3.14 3.14"/>
     </joint>
   </xacro:macro>
